Commit message: Auto-commit on Tue Nov  5 09:30:19 PM CET 2024

File: Babydoll/Produits/Babydoll-01/POC/LearnPyBullet/hexapod_2.urdf (robot description, URDF)
Before this commit: robot hexapod, 25 links, 24 joints
Links:
- added link e1, mass 0.01; collision sphere radius=0.02; visual sphere radius=0.02
- added link e2, mass 0.01; collision sphere radius=0.02; visual sphere radius=0.02
- added link e3, mass 0.01; collision sphere radius=0.02; visual sphere radius=0.02
- added link e4, mass 0.01; collision sphere radius=0.02; visual sphere radius=0.02
- added link e5, mass 0.01; collision sphere radius=0.02; visual sphere radius=0.02
- added link e6, mass 0.01; collision sphere radius=0.02; visual sphere radius=0.02
- link body: mass 0.5 -> 0.01
Joints:
- added joint x1: type fixed, parent d1, child e1, origin xyz=0 0.14 0 rpy=0 0 0
- added joint x2: type fixed, parent d2, child e2, origin xyz=0 0.14 0 rpy=0 0 0
- added joint x3: type fixed, parent d3, child e3, origin xyz=0 0.14 0 rpy=0 0 0
- added joint x4: type fixed, parent d4, child e4, origin xyz=0 0.14 0 rpy=0 0 0
- added joint x5: type fixed, parent d5, child e5, origin xyz=0 0.14 0 rpy=0 0 0
- added joint x6: type fixed, parent d6, child e6, origin xyz=0 0.14 0 rpy=0 0 0
- joint u1: limit lower=-1.57 upper=1.57 effort=100 velocity=1 -> lower=-1.57 upper=1.57 effort=1000 velocity=1000; type revolute -> continuous
- joint u2: limit lower=-1.57 upper=1.57 effort=100 velocity=1 -> lower=-1.57 upper=1.57 effort=1000 velocity=1000; type revolute -> continuous
- joint u3: limit lower=-1.57 upper=1.57 effort=100 velocity=1 -> lower=-1.57 upper=1.57 effort=1000 velocity=1000; type revolute -> continuous
- joint u4: limit lower=-1.57 upper=1.57 effort=100 velocity=1 -> lower=-1.57 upper=1.57 effort=1000 velocity=1000; type revolute -> continuous
- joint u5: limit lower=-1.57 upper=1.57 effort=100 velocity=1 -> lower=-1.57 upper=1.57 effort=1000 velocity=1000; type revolute -> continuous
- joint u6: limit lower=-1.57 upper=1.57 effort=100 velocity=1 -> lower=-1.57 upper=1.57 effort=1000 velocity=1000; type revolute -> continuous
- joint v1: limit lower=-1.57 upper=1.57 effort=100 velocity=1 -> lower=-1.57 upper=1.57 effort=1000 velocity=1000; type revolute -> continuous
- joint v2: limit lower=-1.57 upper=1.57 effort=100 velocity=1 -> lower=-1.57 upper=1.57 effort=1000 velocity=1000; type revolute -> continuous
- joint v3: limit lower=-1.57 upper=1.57 effort=100 velocity=1 -> lower=-1.57 upper=1.57 effort=1000 velocity=1000; type revolute -> continuous
- joint v4: limit lower=-1.57 upper=1.57 effort=100 velocity=1 -> lower=-1.57 upper=1.57 effort=1000 velocity=1000; type revolute -> continuous
- joint v5: limit lower=-1.57 upper=1.57 effort=100 velocity=1 -> lower=-1.57 upper=1.57 effort=1000 velocity=1000; type revolute -> continuous
- joint v6: limit lower=-1.57 upper=1.57 effort=100 velocity=1 -> lower=-1.57 upper=1.57 effort=1000 velocity=1000; type revolute -> continuous
- joint w1: limit lower=-1.57 upper=1.57 effort=100 velocity=1 -> lower=-3.14159 upper=1.57 effort=1000 velocity=1000; type revolute -> continuous
- joint w2: limit lower=-1.57 upper=1.57 effort=100 velocity=1 -> lower=-3.14159 upper=1.57 effort=1000 velocity=1000; type revolute -> continuous
- joint w3: limit lower=-1.57 upper=1.57 effort=100 velocity=1 -> lower=-3.14159 upper=1.57 effort=1000 velocity=1000; type revolute -> continuous
- joint w4: limit lower=-1.57 upper=1.57 effort=100 velocity=1 -> lower=-3.14159 upper=1.57 effort=1000 velocity=1000; type revolute -> continuous
- joint w5: limit lower=-1.57 upper=1.57 effort=100 velocity=1 -> lower=-3.14159 upper=1.57 effort=1000 velocity=1000; type revolute -> continuous
- joint w6: limit lower=-1.57 upper=1.57 effort=100 velocity=1 -> lower=-3.14159 upper=1.57 effort=1000 velocity=1000; type revolute -> continuous
